File: CAN_T.kicad_sch (KiCad schematic)
At the start: 16 parts, among them J10 BM02B-GHS-TBT, U10 MAX7375AXR805

Commit message: Imported updated files from office verison of this project
Connections:
- net CAN+: now reaches C26.2, D2.1 (K), J10.1 (Pin_1), R15.1, U?.4 (CANH)
- net CAN-: now reaches C27.2, D2.2 (K), J10.2 (Pin_2), R16.2, U?.3 (CANL)
Other:
- company: (none) -> Toofon Inc.
Changed lines of the file:
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@@
   (title_block
     (title "Test Stand Power Monitor")
-    (date "2023-06-05")
+    (date "2023-08-08")
     (rev "1.0")
+    (company "Toofon Inc.")
     (comment 1 "Ed Katynski")
     (comment 2 "(PENDING REVIEW)")
@@
     (effects (font (size 1.27 1.27)) (justify left bottom))
   )
+  (label "CAN-" (at 218.44 91.44 0) (fields_autoplaced)
+    (effects (font (size 1.27 1.27)) (justify left bottom))
+  )
+  (label "CAN+" (at 218.44 88.9 0) (fields_autoplaced)
+    (effects (font (size 1.27 1.27)) (justify left bottom))
+  )
