File: Voltage.kicad_sch (KiCad schematic)
At the start: 7 parts, among them J7 560020-0230

Commit message: Imported updated files from office verison of this project
Other:
- company: (none) -> Toofon Inc.
Changed lines of the file:
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@@
   (title_block
     (title "Test Stand Power Monitor")
-    (date "2023-06-05")
+    (date "2023-08-08")
     (rev "1.0")
+    (company "Toofon Inc.")
     (comment 1 "Ed Katynski")
     (comment 2 "(PENDING REVIEW)")
