File: Test-Stand-Power-Monitor.kicad_pcb (KiCad board)
At the start: 2 copper layers, 56.3 x 68.4 mm, 70 parts, among them J1 560020-0330, J10 BM02B-GHS-TBT, J2 Conn_01x02_Pin, J3 1715721, J4 Conn_01x03_Pin, J5 BM03B-GHS-TBT, J6 BM02B-GHS-TBT, J7 560020-0230, J8 BM04B-GHS-TBT, J9 BM03B-GHS-TBT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

Commit message: Imported updated files from office verison of this project
Connections:
- net Net-(J10-Pin_1) renamed /CAN Transceiver/CAN+
- net Net-(J10-Pin_2) renamed /CAN Transceiver/CAN-
Routing:
- net GND: vias 275 -> 274
- added copper zone on In1.Cu, net GND
- added copper zone on In2.Cu, net GND
Other:
- copper layers 2 -> 4
- board text added: "NUM: . DATE:"
- board text removed: "NUM: DATE:"

Commit message: Slight 3.3V power trace movement for improved ground pour
Routing:
- net +3.3V: track 101.3 -> 102.2 mm
- net +5V: track 155.3 -> 156.1 mm
